File: Hardware/RevC/AriCalculator-RevC-Display.sch (KiCad schematic (older format))
At the start: 33 parts, among them IC4 MCP1643

Commit message: work in progress
Parts:
- C13: value 1uf -> 1uF
Changed lines of the file:
@@
 Sheet 4 6
 Title "Display"
-Date "25 nov 2014"
+Date "4 dec 2014"
 Rev "RevC"
 Comp "Dirk Heisswolf"
@@
 P 3100 3600
 F 0 "C13" H 3100 3700 40  0000 L CNN
-F 1 "1uf" H 3106 3515 40  0000 L CNN
+F 1 "1uF" H 3106 3515 40  0000 L CNN
 F 2 "~" H 3138 3450 30  0000 C CNN
 F 3 "~" H 3100 3600 60  0000 C CNN
