File: Hardware/RevC/AriCalculator-RevC-MCU.sch (KiCad schematic (older format))
At the start: 15 parts, among them CON1 BDM, CON2 SPI, IC1 MC9S12G

Commit message: work in progress
Connections:
- net 3V3: now also R1.1, R2.1; no longer LED1.2 (K), LED2.2 (K)
- net at IC1.4 (PE0/EXTAL): now also LED1.1 (A); no longer R1.2
- net at IC1.6 (PE1/XTAL): now also LED2.1 (A); no longer R2.2
- new net: LED1.2 (K), R1.2
- new net: LED2.2 (K), R2.2
Other:
- moved on the sheet: LED1, LED2, R1, R2
Changed lines of the file:
@@
 Sheet 6 6
 Title "MCU"
-Date "15 nov 2014"
+Date "25 nov 2014"
 Rev "RevC"
 Comp "Dirk Heisswolf"
@@
 L R R1
 U 1 1 544FF846
-P 2000 2200
-F 0 "R1" V 2080 2200 40  0000 C CNN
-F 1 "120" V 2007 2201 40  0000 C CNN
-F 2 "~" V 1930 2200 30  0000 C CNN
-F 3 "~" H 2000 2200 30  0000 C CNN
-	1    2000 2200
+P 1550 2200
+F 0 "R1" V 1630 2200 40  0000 C CNN
+F 1 "120" V 1557 2201 40  0000 C CNN
+F 2 "~" V 1480 2200 30  0000 C CNN
+F 3 "~" H 1550 2200 30  0000 C CNN
+	1    1550 2200
 	0    -1   -1   0
 $EndComp
@@
 L R R2
 U 1 1 544FF855
-P 2000 2400
-F 0 "R2" V 2080 2400 40  0000 C CNN
-F 1 "120" V 2007 2401 40  0000 C CNN
-F 2 "~" V 1930 2400 30  0000 C CNN
-F 3 "~" H 2000 2400 30  0000 C CNN
-	1    2000 2400
+P 1550 2400
+F 0 "R2" V 1630 2400 40  0000 C CNN
+F 1 "120" V 1557 2401 40  0000 C CNN
+F 2 "~" V 1480 2400 30  0000 C CNN
+F 3 "~" H 1550 2400 30  0000 C CNN
+	1    1550 2400
 	0    -1   -1   0
 $EndComp
@@
 L LED LED1
 U 1 1 544FF88C
-P 1500 2200
-F 0 "LED1" H 1500 2300 50  0000 C CNN
-F 1 "GREEN" H 1300 2150 50  0000 C CNN
-F 2 "~" H 1500 2200 60  0000 C CNN
-F 3 "~" H 1500 2200 60  0000 C CNN
-	1    1500 2200
+P 2050 2200
+F 0 "LED1" H 2050 2300 50  0000 C CNN
+F 1 "GREEN" H 1850 2150 50  0000 C CNN
+F 2 "~" H 2050 2200 60  0000 C CNN
+F 3 "~" H 2050 2200 60  0000 C CNN
+	1    2050 2200
 	-1   0    0    -1
 $EndComp
@@
 L LED LED2
 U 1 1 544FF89B
-P 1500 2400
-F 0 "LED2" H 1500 2500 50  0000 C CNN
-F 1 "RED" H 1350 2350 50  0000 C CNN
-F 2 "~" H 1500 2400 60  0000 C CNN
-F 3 "~" H 1500 2400 60  0000 C CNN
-	1    1500 2400
+P 2050 2400
+F 0 "LED2" H 2050 2500 50  0000 C CNN
+F 1 "RED" H 1900 2350 50  0000 C CNN
+F 2 "~" H 2050 2400 60  0000 C CNN
+F 3 "~" H 2050 2400 60  0000 C CNN
+	1    2050 2400
 	-1   0    0    -1
 $EndComp
@@
 	2800 2400 2250 2400
 Wire Wire Line
-	1750 2200 1700 2200
-Wire Wire Line
-	1750 2400 1700 2400
+	1850 2200 1800 2200
+Wire Wire Line
+	1850 2400 1800 2400
 Wire Wire Line
 	1300 2200 1250 2200

Commit message: work in progress
Parts:
- C1: value 100nf -> 100nF
Changed lines of the file:
@@
 Sheet 6 6
 Title "MCU"
-Date "25 nov 2014"
+Date "4 dec 2014"
 Rev "RevC"
 Comp "Dirk Heisswolf"
@@
 $EndComp
 $Comp
-L GND #PWR025
+L GND #PWR026
 U 1 1 544FF350
 P 4900 1400
-F 0 "#PWR025" H 4900 1400 30  0001 C CNN
+F 0 "#PWR026" H 4900 1400 30  0001 C CNN
 F 1 "GND" H 4900 1330 30  0001 C CNN
 F 2 "" H 4900 1400 60  0000 C CNN
@@
 P 4700 1350
 F 0 "C1" H 4700 1450 40  0000 L CNN
-F 1 "100nf" H 4706 1265 40  0000 L CNN
+F 1 "100nF" H 4706 1265 40  0000 L CNN
 F 2 "~" H 4738 1200 30  0000 C CNN
 F 3 "~" H 4700 1350 60  0000 C CNN
@@
 $EndComp
 $Comp
-L GND #PWR026
+L GND #PWR027
 U 1 1 544FF410
 P 2300 2600
-F 0 "#PWR026" H 2300 2600 30  0001 C CNN
+F 0 "#PWR027" H 2300 2600 30  0001 C CNN
 F 1 "GND" H 2300 2530 30  0001 C CNN
 F 2 "" H 2300 2600 60  0000 C CNN
@@
 $EndComp
 $Comp
-L GND #PWR027
+L GND #PWR028
 U 1 1 544FF75E
 P 1300 3200
-F 0 "#PWR027" H 1300 3200 30  0001 C CNN
+F 0 "#PWR028" H 1300 3200 30  0001 C CNN
 F 1 "GND" H 1300 3130 30  0001 C CNN
 F 2 "" H 1300 3200 60  0000 C CNN
@@
 KEYPAD_ROW_F
 $Comp
-L +BATT #PWR028
+L +BATT #PWR029
 U 1 1 544FFB66
 P 5050 2900
-F 0 "#PWR028" H 5050 2850 20  0001 C CNN
+F 0 "#PWR029" H 5050 2850 20  0001 C CNN
 F 1 "+BATT" V 5050 3050 30  0000 C CNN
 F 2 "" H 5050 2900 60  0000 C CNN
@@
 	4350 3650 4350 3550
 $Comp
-L GND #PWR029
+L GND #PWR030
 U 1 1 545A5D88
 P 1300 4200
-F 0 "#PWR029" H 1300 4200 30  0001 C CNN
+F 0 "#PWR030" H 1300 4200 30  0001 C CNN
 F 1 "GND" H 1300 4130 30  0001 C CNN
 F 2 "~" H 1300 4200 60  0000 C CNN
