File: Hardware/RevC/AriCalculator-RevC-UART.sch (KiCad schematic (older format))
At the start: 15 parts, among them CON3 USB-MINI-B, IC3 FT232RL

Commit message: work in progress
Parts:
- added C21: 100nF, ~, symbol C
Connections:
- net GND: now also C21.2
- net at C18.1, IC3.17 (3V3OUT), IC3.4 (VCCIO)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: now also C21.1
Other:
- moved on the sheet: R11, R12
Changed lines of the file:
@@
 Sheet 5 6
 Title "UART"
-Date "25 nov 2014"
+Date "4 dec 2014"
 Rev "RevC"
 Comp "Dirk Heisswolf"
@@
 L R R11
 U 1 1 54503F24
-P 3650 2650
-F 0 "R11" V 3730 2650 40  0000 C CNN
-F 1 "4K7" V 3657 2651 40  0000 C CNN
-F 2 "~" V 3580 2650 30  0000 C CNN
-F 3 "~" H 3650 2650 30  0000 C CNN
-	1    3650 2650
+P 3450 2650
+F 0 "R11" V 3530 2650 40  0000 C CNN
+F 1 "4K7" V 3457 2651 40  0000 C CNN
+F 2 "~" V 3380 2650 30  0000 C CNN
+F 3 "~" H 3450 2650 30  0000 C CNN
+	1    3450 2650
 	-1   0    0    -1
 $EndComp
@@
 L R R12
 U 1 1 54503F33
-P 3650 3250
-F 0 "R12" V 3730 3250 40  0000 C CNN
-F 1 "10K" V 3657 3251 40  0000 C CNN
-F 2 "~" V 3580 3250 30  0000 C CNN
-F 3 "~" H 3650 3250 30  0000 C CNN
-	1    3650 3250
+P 3450 3250
+F 0 "R12" V 3530 3250 40  0000 C CNN
+F 1 "10K" V 3457 3251 40  0000 C CNN
+F 2 "~" V 3380 3250 30  0000 C CNN
+F 3 "~" H 3450 3250 30  0000 C CNN
+	1    3450 3250
 	-1   0    0    -1
 $EndComp
@@
 L GND #PWR021
 U 1 1 54503FB1
-P 3650 3550
-F 0 "#PWR021" H 3650 3550 30  0001 C CNN
-F 1 "GND" H 3650 3480 30  0001 C CNN
-F 2 "" H 3650 3550 60  0000 C CNN
-F 3 "" H 3650 3550 60  0000 C CNN
-	1    3650 3550
+P 3450 3550
+F 0 "#PWR021" H 3450 3550 30  0001 C CNN
+F 1 "GND" H 3450 3480 30  0001 C CNN
+F 2 "" H 3450 3550 60  0000 C CNN
+F 3 "" H 3450 3550 60  0000 C CNN
+	1    3450 3550
 	1    0    0    -1
 $EndComp
@@
 	2600 2600 2600 2700
 Wire Wire Line
-	3850 3100 4000 3100
+	3650 3100 4000 3100
 Wire Wire Line
 	3850 3500 3850 3550
@@
 	4000 1850 3850 1850
 Wire Wire Line
-	3650 3500 3650 3550
-Wire Wire Line
-	3650 2900 3650 3000
+	3450 3500 3450 3550
+Wire Wire Line
+	3450 2900 3450 3000
 Wire Wire Line
 	3400 1950 4000 1950
 Wire Wire Line
-	3650 1950 3650 2400
-Connection ~ 3650 2950
+	3450 1950 3450 2400
+Connection ~ 3450 2950
 Wire Wire Line
 	4000 2300 2600 2300
@@
 	3900 2600 3900 2950
 Wire Wire Line
-	3900 2950 3550 2950
-Wire Wire Line
 	2600 2200 2600 2150
 Wire Wire Line
@@
 Wire Wire Line
 	2600 1150 2600 2000
-Connection ~ 3650 1950
+Connection ~ 3450 1950
 Wire Wire Line
 	5850 2900 6000 2900
@@
 Wire Wire Line
 	6100 2200 5850 2200
-Text HLabel 3550 2950 0    60   UnSpc ~ 0
+Text HLabel 3350 2950 0    60   UnSpc ~ 0
 VUSB_SENSE
 Text Label 2650 2300 0    60   ~ 0
@@
 Wire Wire Line
 	1500 2600 1450 2600
+$Comp
+L C C21
+U 1 1 54805555
+P 3650 3300
+F 0 "C21" H 3650 3400 40  0000 L CNN
+F 1 "100nF" H 3656 3215 40  0000 L CNN
+F 2 "~" H 3688 3150 30  0000 C CNN
+F 3 "~" H 3650 3300 60  0000 C CNN
+	1    3650 3300
+	1    0    0    -1
+$EndComp
+Connection ~ 3850 3100
+$Comp
+L GND #PWR025
+U 1 1 548055AD
+P 3650 3550
+F 0 "#PWR025" H 3650 3550 30  0001 C CNN
+F 1 "GND" H 3650 3480 30  0001 C CNN
+F 2 "~" H 3650 3550 60  0000 C CNN
+F 3 "~" H 3650 3550 60  0000 C CNN
+	1    3650 3550
+	1    0    0    -1
+$EndComp
+Wire Wire Line
+	3650 3500 3650 3550
+Wire Wire Line
+	3900 2950 3350 2950
 $EndSCHEMATC
