File: Hardware/RevC/AriCalculator-RevC.kicad_pcb (KiCad board)
At the start: 2 copper layers, 76.2 x 147.3 mm, 126 parts, among them CON1 BDM, CON2 SPI, CON3 USB-MINI-B, IC1 MC9S12G, IC2 MCP1640, IC3 FT232RL, IC4 MCP1643, SW1 POWER SWITCH

Commit message: work in progress
Parts:
- removed the spark_gap_pad_0.8 at (141.1, 111.3)
- removed the spark_gap_pad_0.8 at (141.2, 110.3)
- added ?: , VIA, B.Cu at (112.0, 119.4)
- added ?: , VIA, F.Cu at (104.2, 113.5)
- added ?: , VIA, F.Cu at (103.3, 110.7)
- added ?: , VIA, F.Cu at (105.8, 118.4)
- added ?: , VIA, F.Cu at (87.4, 107.7)
- added ?: , VIA, F.Cu at (111.4, 103.1)
- added ?: , VIA, F.Cu at (101.6, 115.6)
- added ?: , VIA, F.Cu at (112.6, 103.1)
- added ?: , VIA, F.Cu at (129.3, 98.4)
- added ?: , VIA, F.Cu at (84.1, 99.7)
- added ?: , VIA, F.Cu at (84.1, 98.5)
- added ?: , VIA, F.Cu at (113.8, 103.1)
- added ?: , VIA, B.Cu at (109.8, 119.3)
- added spark_gap_pad_0.6: SG, spark_gap_pad_0.6, B.Cu at (85.0, 98.5)
- added spark_gap_pad_0.6: SG, spark_gap_pad_0.6, B.Cu at (128.4, 98.4)
- added spark_gap_pad_0.6: SG, spark_gap_pad_0.6, B.Cu at (128.4, 97.8)
- added spark_gap_pad_0.6: SG, spark_gap_pad_0.6, B.Cu at (128.4, 97.2)
- added spark_gap_pad_0.6: SG, spark_gap_pad_0.6, B.Cu at (128.4, 99.0)
- added spark_gap_pad_0.6: SG, spark_gap_pad_0.6, B.Cu at (128.4, 99.6)
- added spark_gap_pad_0.6: SG, spark_gap_pad_0.6, B.Cu at (85.0, 97.9)
- added spark_gap_pad_0.6: SG, spark_gap_pad_0.6, B.Cu at (85.0, 99.1)
- added spark_gap_pad_0.6: SG, spark_gap_pad_0.6, B.Cu at (85.0, 99.7)
- added spark_gap_pad_0.6: SG, spark_gap_pad_0.6, B.Cu at (85.0, 100.3)
- added spark_gap_pad_0.6: SG, spark_gap_pad_0.6, B.Cu at (85.0, 100.9)
- added spark_gap_pad_0.6: SG, spark_gap_pad_0.6, B.Cu at (85.0, 97.3)
- added spark_gap_pad_0.6: SG, spark_gap_pad_0.6, B.Cu at (85.0, 96.7)
- added spark_gap_pad_0.6: SG, spark_gap_pad_0.6, B.Cu at (85.0, 96.1)
- added spark_gap_pad_1.0: SG, spark_gap_pad_1.0, B.Cu at (129.0, 108.6)
- added spark_gap_pad_1.0: SG, spark_gap_pad_1.0, B.Cu at (129.0, 107.6)
- added spark_gap_pad_1.0: SG, spark_gap_pad_1.0, B.Cu at (129.0, 109.6)
- added spark_gap_pad_1.0: SG, spark_gap_pad_1.0, B.Cu at (82.5, 103.3)
- added spark_gap_pad_1.0: SG, spark_gap_pad_1.0, B.Cu at (83.5, 103.3)
- added spark_gap_pad_1.0: SG, spark_gap_pad_1.0, B.Cu at (81.5, 103.3)
- added spark_gap_pad_1.0: SG, spark_gap_pad_1.0, B.Cu at (128.4, 101.6)
- added spark_gap_pad_1.0: SG, spark_gap_pad_1.0, B.Cu at (128.4, 100.6)
- added spark_gap_pad_1.0: SG, spark_gap_pad_1.0, B.Cu at (128.4, 102.6)
- C19, C20, IC4, L2, R1, R14, R2: moved to B.Cu
- LED20, LED21: value IR -> BACKLIGHT; footprint led_5mm_bend -> Led_1206; moved to F.Cu
- moved LED4 96.8 mm to (81.6, 94.2)
- moved LED5 90.2 mm to (94.1, 94.2), turned to 180 degrees
- moved LED14 89.7 mm to (81.6, 121.0)
- moved LED9 85.9 mm to (79.8, 107.6), turned to 270 degrees
- moved LED6 78.9 mm to (106.7, 94.2)
- moved LED19 77.1 mm to (93.3, 111.8), turned to 180 degrees
- moved LED10 72.4 mm to (93.3, 103.4), turned to 180 degrees
- moved LED7 70.1 mm to (119.3, 94.2), turned to 180 degrees
- moved LED15 67.7 mm to (94.1, 121.0), turned to 180 degrees
- moved LED16 66.2 mm to (106.7, 121.0)
- moved LED8 63.0 mm to (131.8, 94.2)
- moved LED11 55.0 mm to (106.7, 103.4)
- moved LED17 52.7 mm to (119.3, 121.0), turned to 180 degrees
- moved LED12 50.9 mm to (120.0, 103.4), turned to 180 degrees
- moved C19 49.4 mm to (136.4, 129.8)
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Routing:
- net N-0000068: track 0.00 -> 147.0 mm, vias 0 -> 2
- net N-0000067: track 0.00 -> 127.7 mm
- net 3V3: track 5.17 -> 114.5 mm
- net N-0000034: track 0.00 -> 59.6 mm, vias 0 -> 2
- net N-0000031: track 0.00 -> 55.8 mm, vias 0 -> 2
- net /Display/DISPLAY_SS: track 0.00 -> 53.8 mm, vias 0 -> 2
- net N-0000030: track 0.00 -> 49.4 mm, vias 0 -> 2
- net N-0000026: track 0.00 -> 49.3 mm, vias 0 -> 2
- net N-0000045: track 0.00 -> 48.4 mm, vias 0 -> 2
- net /Display/DISPLAY_RESET: track 0.00 -> 46.1 mm, vias 0 -> 1
- net N-0000033: track 0.00 -> 43.6 mm, vias 0 -> 2
- net /Display/DISPLAY_A0: track 0.00 -> 42.5 mm, vias 0 -> 1
- net /Display/DISPLAY_MOSI: track 0.00 -> 42.4 mm, vias 0 -> 1
- net /Display/DISPLAY_SCK: track 0.00 -> 41.0 mm, vias 0 -> 1
- net +BATT: track 0.00 -> 36.4 mm
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
Commit message: work in progress
Parts:
- removed the ? at (105.8, 118.4)
- added spark_gap_pad_0.6: SG, spark_gap_pad_0.6, B.Cu at (135.0, 117.5)
- added spark_gap_pad_0.6: SG, spark_gap_pad_0.6, B.Cu at (135.0, 116.9)
- added spark_gap_pad_0.6: SG, spark_gap_pad_0.6, B.Cu at (135.0, 118.1)
- SW1: moved to B.Cu
- moved LED1 66.1 mm to (72.0, 131.8)
- moved LED2 66.0 mm to (74.1, 131.8)
- moved R1 43.1 mm to (72.0, 131.8), turned to 90 degrees
- moved R2 41.4 mm to (74.1, 131.8), turned to 90 degrees
- moved ? 5.89 mm to (103.6, 107.7)
- moved ? 4.12 mm to (103.7, 106.6)
- moved ? 3.38 mm to (110.0, 115.9)
- turned SW1 to 270 degrees
Connections:
- LED1 pad 1: N-0000028 -> N-0000044
- LED1 pad 2: 3V3 -> N-0000028
- LED2 pad 1: N-0000035 -> N-0000043
- LED2 pad 2: 3V3 -> N-0000035
- R1 pad 1: N-0000028 -> 3V3
- R1 pad 2: N-0000044 -> N-0000028
- R2 pad 1: N-0000035 -> 3V3
- R2 pad 2: N-0000043 -> N-0000035
- SW1 pad 1: N-0000093 -> GND
- SW1 pad 3: GND -> N-0000093
Routing:
- net N-0000068: track 147.0 -> 236.8 mm, vias 2 -> 5
- net 3V3: track 114.5 -> 189.0 mm
- net N-0000067: track 127.7 -> 182.3 mm, vias 0 -> 3
- net N-0000044: track 0.00 -> 50.7 mm, vias 0 -> 3
- net N-0000043: track 0.00 -> 49.0 mm, vias 0 -> 1
- net +BATT: track 36.4 -> 82.4 mm, vias 0 -> 2
- net /Display/DISPLAY_BACKLIGHT: track 0.00 -> 29.7 mm, vias 0 -> 2
- net GND: track 29.1 -> 13.7 mm
- net /MCU/VUSB_SENSE: track 41.1 -> 42.1 mm
- net /Keypad/KEYPAD_ROW_A: track 130.3 -> 129.7 mm
- net N-0000035: track 0.00 -> 0.19 mm, vias 0 -> 1
- net N-0000028: track 0.00 -> 0.19 mm, vias 0 -> 1
- net N-0000051: track 11.9 -> 11.8 mm, vias 0 -> 2

Commit message: work in progress
Parts:
- added ?: , VIA, F.Cu at (117.3, 95.6)
- added ?: , VIA, F.Cu at (128.4, 100.0)
- added ?: , VIA, F.Cu at (109.4, 97.3)
- added ?: , VIA, F.Cu at (109.4, 96.0)
- added ?: , VIA, F.Cu at (109.4, 98.5)
- added ?: , VIA, F.Cu at (110.0, 99.7)
- added ?: , VIA, F.Cu at (110.1, 101.0)
- added ?: , VIA, F.Cu at (105.9, 101.0)
- added ?: , VIA, F.Cu at (107.5, 99.7)
- added ?: , VIA, F.Cu at (105.9, 98.5)
- added ?: , VIA, F.Cu at (105.9, 96.0)
- added ?: , VIA, F.Cu at (107.5, 97.3)
- added ?: , VIA, F.Cu at (119.0, 93.8)
- added ?: , VIA, F.Cu at (102.0, 96.0)
- added ?: , VIA, F.Cu at (104.0, 97.3)
- added ?: , VIA, F.Cu at (102.0, 97.3)
- added ?: , VIA, F.Cu at (99.6, 96.0)
- added ?: , VIA, F.Cu at (100.8, 97.3)
- added ?: , VIA, F.Cu at (100.8, 95.1)
- added ?: , VIA, F.Cu at (99.6, 97.3)
- added ?: , VIA, F.Cu at (96.0, 96.0)
- added ?: , VIA, F.Cu at (97.1, 97.3)
- added ?: , VIA, F.Cu at (98.4, 97.3)
- added ?: , VIA, F.Cu at (122.7, 95.2)
- added ?: , VIA, F.Cu at (103.3, 95.1)
- added ?: , VIA, F.Cu at (98.4, 95.1)
- added ?: , VIA, F.Cu at (102.0, 107.7)
- added ?: , VIA, F.Cu at (100.8, 107.7)
- added ?: , VIA, F.Cu at (99.6, 107.7)
- added ?: , VIA, F.Cu at (96.0, 101.0)
- added ?: , VIA, F.Cu at (98.4, 107.7)
- added ?: , VIA, F.Cu at (115.2, 97.3)
- added ?: , VIA, F.Cu at (98.4, 98.5)
- added ?: , VIA, F.Cu at (103.3, 98.5)
- added ?: , VIA, F.Cu at (135.4, 107.1)
- added ?: , VIA, F.Cu at (98.4, 99.7)
- added ?: , VIA, F.Cu at (97.1, 99.7)
- added ?: , VIA, F.Cu at (96.0, 98.5)
- added ?: , VIA, F.Cu at (135.8, 110.7)
- added ?: , VIA, F.Cu at (79.3, 103.1)
- added ?: , VIA, F.Cu at (73.7, 134.6)
- added ?: , VIA, F.Cu at (141.4, 111.4)
- added ?: , VIA, F.Cu at (72.6, 109.5)
- added ?: , VIA, F.Cu at (122.2, 90.2)
- added ?: , VIA, F.Cu at (112.2, 120.7)
- added ?: , VIA, F.Cu at (131.1, 107.0)
- added ?: , VIA, F.Cu at (112.5, 97.3)
- added ?: , VIA, F.Cu at (105.8, 114.5)
- added ?: , VIA, F.Cu at (100.8, 120.7)
- added ?: , VIA, F.Cu at (100.7, 128.5)
- added ?: , VIA, F.Cu at (111.3, 98.5)
- added ?: , VIA, F.Cu at (138.5, 110.7)
- added ?: , VIA, F.Cu at (90.5, 104.7)
- added ?: , VIA, F.Cu at (113.8, 96.0)
- added ?: , VIA, F.Cu at (81.5, 102.7)
- added ?: , VIA, F.Cu at (99.6, 128.5)
- added ?: , VIA, F.Cu at (132.1, 110.0)
- added ?: , VIA, F.Cu at (99.6, 121.0)
- added ?: , VIA, F.Cu at (74.3, 121.9)
- added ?: , VIA, F.Cu at (78.8, 122.3)
- added ?: , VIA, F.Cu at (77.3, 120.2)
- added ?: , VIA, F.Cu at (73.0, 129.7)
- added ?: , VIA, F.Cu at (106.4, 130.3)
- added ?: , VIA, F.Cu at (72.6, 198.9)
- added ?: , VIA, F.Cu at (87.0, 119.7)
- added ?: , VIA, F.Cu at (83.5, 123.2)
- added ?: , VIA, F.Cu at (73.7, 165.1)
- added ?: , VIA, F.Cu at (134.4, 111.9)
- added ?: , VIA, F.Cu at (73.7, 154.9)
- added ?: , VIA, F.Cu at (116.2, 120.8)
- added ?: , VIA, F.Cu at (104.0, 130.3)
- added ?: , VIA, F.Cu at (74.3, 113.0)
- added ?: , VIA, F.Cu at (73.2, 117.4)
- added ?: , VIA, F.Cu at (108.6, 128.6)
- added ?: , VIA, F.Cu at (105.3, 128.6)
- added ?: , VIA, F.Cu at (103.3, 120.8)
- added ?: , VIA, F.Cu at (94.4, 116.6)
- added ?: , VIA, F.Cu at (99.5, 118.0)
- added ?: , VIA, F.Cu at (134.4, 116.8)
- added ?: , VIA, F.Cu at (105.9, 118.3)
- added ?: , VIA, F.Cu at (93.8, 120.9)
- added ?: , VIA, F.Cu at (91.2, 118.7)
- added ?: , VIA, F.Cu at (139.7, 195.6)
- added ?: , VIA, F.Cu at (134.6, 200.7)
- added ?: , VIA, F.Cu at (72.6, 80.5)
- added ?: , VIA, F.Cu at (72.6, 88.6)
- added ?: , VIA, F.Cu at (140.5, 117.5)
- added ?: , VIA, F.Cu at (73.7, 185.4)
- added ?: , VIA, F.Cu at (73.7, 195.6)
- added ?: , VIA, F.Cu at (129.2, 122.3)
- added ?: , VIA, F.Cu at (132.9, 92.0)
- added ?: , VIA, F.Cu at (139.7, 185.4)
- added ?: , VIA, F.Cu at (139.7, 209.6)
- added ?: , VIA, F.Cu at (73.7, 144.8)
- added ?: , VIA, F.Cu at (73.7, 175.3)
- added ?: , VIA, F.Cu at (139.7, 134.6)
- added ?: , VIA, F.Cu at (139.7, 144.8)
- added ?: , VIA, F.Cu at (139.7, 154.9)
- added ?: , VIA, F.Cu at (139.7, 165.1)
- added ?: , VIA, F.Cu at (139.7, 175.3)
- added ?: , VIA, F.Cu at (130.9, 122.7)
- added ?: , VIA, F.Cu at (128.4, 109.5)
- added ?: , VIA, F.Cu at (110.1, 107.7)
- added ?: , VIA, F.Cu at (113.8, 110.8)
- added ?: , VIA, F.Cu at (93.5, 83.5)
- added ?: , VIA, F.Cu at (93.2, 112.3)
- added ?: , VIA, F.Cu at (115.1, 109.5)
- added ?: , VIA, F.Cu at (107.1, 112.7)
- added ?: , VIA, F.Cu at (109.4, 109.5)
- added ?: , VIA, F.Cu at (119.2, 109.5)
- added ?: , VIA, F.Cu at (104.0, 107.7)
- added ?: , VIA, F.Cu at (126.5, 92.0)
- added ?: , VIA, F.Cu at (132.2, 116.8)
- added ?: , VIA, F.Cu at (95.8, 92.8)
- added ?: , VIA, F.Cu at (105.9, 109.5)
- added ?: , VIA, F.Cu at (103.3, 109.7)
- added ?: , VIA, F.Cu at (107.5, 107.7)
- added ?: , VIA, F.Cu at (117.3, 107.7)
- added ?: , VIA, F.Cu at (127.1, 109.5)
- added ?: , VIA, F.Cu at (86.7, 115.3)
- added ?: , VIA, F.Cu at (113.8, 116.2)
- added ?: , VIA, F.Cu at (112.6, 107.7)
- added ?: , VIA, F.Cu at (85.7, 118.7)
- added ?: , VIA, F.Cu at (134.4, 118.2)
- added ?: , VIA, F.Cu at (112.6, 109.5)
- added ?: , VIA, F.Cu at (112.6, 112.0)
- added ?: , VIA, F.Cu at (125.8, 107.7)
- added ?: , VIA, F.Cu at (109.9, 111.3)
- added ?: , VIA, F.Cu at (113.8, 107.7)
- added ?: , VIA, F.Cu at (111.4, 113.2)
- added ?: , VIA, F.Cu at (129.3, 107.6)
- added ?: , VIA, F.Cu at (127.1, 106.0)
- added ?: , VIA, F.Cu at (111.4, 110.5)
- added ?: , VIA, F.Cu at (89.0, 115.3)
- added ?: , VIA, F.Cu at (122.0, 122.7)
- added ?: , VIA, F.Cu at (111.4, 107.7)
- added ?: , VIA, F.Cu at (84.5, 117.5)
- added ?: , VIA, F.Cu at (88.7, 119.8)
- added ?: , VIA, F.Cu at (122.9, 88.5)
- added ?: , VIA, F.Cu at (112.6, 116.3)
- added ?: , VIA, F.Cu at (94.5, 118.5)
- added ?: , VIA, F.Cu at (113.8, 118.1)
- added ?: , VIA, F.Cu at (122.7, 109.5)
- added ?: , VIA, F.Cu at (126.8, 130.3)
- added ?: , VIA, F.Cu at (120.8, 107.7)
- added ?: , VIA, F.Cu at (129.2, 116.8)
- added ?: , VIA, F.Cu at (138.6, 128.8)
- added ?: , VIA, F.Cu at (138.7, 126.7)
- added ?: , VIA, F.Cu at (139.1, 124.6)
- added ?: , VIA, F.Cu at (104.7, 122.3)
- added ?: , VIA, F.Cu at (131.6, 125.2)
- added ?: , VIA, F.Cu at (128.6, 127.4)
- added ?: , VIA, F.Cu at (136.0, 126.7)
- added ?: , VIA, F.Cu at (132.3, 128.6)
- added ?: , VIA, F.Cu at (140.7, 80.5)
- added ?: , VIA, F.Cu at (137.8, 118.8)
- added ?: , VIA, F.Cu at (120.2, 122.3)
- added ?: , VIA, F.Cu at (106.5, 125.0)
- added ?: , VIA, F.Cu at (140.7, 88.6)
- added ?: , VIA, F.Cu at (99.6, 99.7)
- added ?: , VIA, F.Cu at (108.2, 122.3)
- added ?: , VIA, F.Cu at (141.3, 124.6)
- added ?: , VIA, F.Cu at (143.9, 122.3)
- added ?: , VIA, F.Cu at (100.8, 98.5)
- added ?: , VIA, F.Cu at (100.8, 99.7)
- added ?: , VIA, F.Cu at (99.6, 98.5)
- added ?: , VIA, F.Cu at (102.0, 99.7)
- added ?: , VIA, F.Cu at (114.7, 120.8)
- added ?: , VIA, F.Cu at (104.0, 99.7)
- added ?: , VIA, F.Cu at (102.0, 98.5)
- added ?: , VIA, F.Cu at (107.1, 120.4)
- added ?: , VIA, F.Cu at (118.5, 118.2)
- added ?: , VIA, F.Cu at (116.7, 116.8)
- added ?: , VIA, F.Cu at (125.8, 116.8)
- added ?: , VIA, F.Cu at (120.1, 116.8)
- added ?: , VIA, F.Cu at (131.4, 93.8)
- added ?: , VIA, F.Cu at (122.0, 118.2)
- added ?: , VIA, F.Cu at (116.7, 119.4)
- added ?: , VIA, F.Cu at (120.1, 119.4)
- added ?: , VIA, F.Cu at (116.2, 118.2)
- added ?: , VIA, F.Cu at (131.3, 120.1)
- added ?: , VIA, F.Cu at (129.2, 118.2)
- added ?: , VIA, F.Cu at (132.7, 122.3)
- added ?: , VIA, F.Cu at (132.7, 118.2)
- added ?: , VIA, F.Cu at (127.1, 118.2)
- added ?: , VIA, F.Cu at (125.8, 119.4)
- added ?: , VIA, F.Cu at (117.7, 92.8)
- added ?: , VIA, F.Cu at (127.1, 116.8)
- added ?: , VIA, F.Cu at (128.7, 120.1)
- added ?: , VIA, F.Cu at (89.2, 135.6)
- added ?: , VIA, F.Cu at (79.8, 137.6)
- added ?: , VIA, F.Cu at (94.4, 126.5)
- added ?: , VIA, F.Cu at (81.2, 129.9)
- added ?: , VIA, F.Cu at (81.7, 126.6)
- added ?: , VIA, F.Cu at (81.7, 128.2)
- added ?: , VIA, F.Cu at (76.6, 131.6)
- added ?: , VIA, F.Cu at (71.8, 128.7)
- added ?: , VIA, F.Cu at (126.6, 96.9)
- added ?: , VIA, F.Cu at (94.5, 123.2)
- added ?: , VIA, F.Cu at (90.2, 112.3)
- added ?: , VIA, F.Cu at (93.5, 115.0)
- added ?: , VIA, F.Cu at (96.8, 112.7)
- added ?: , VIA, F.Cu at (98.8, 114.2)
- added ?: , VIA, F.Cu at (95.0, 113.2)
- added ?: , VIA, F.Cu at (103.3, 112.7)
- added ?: , VIA, F.Cu at (96.0, 110.2)
- added ?: , VIA, F.Cu at (100.8, 111.0)
- added ?: , VIA, F.Cu at (102.0, 111.0)
- added ?: , VIA, F.Cu at (124.0, 92.0)
- added ?: , VIA, F.Cu at (103.2, 111.0)
- added ?: , VIA, F.Cu at (98.4, 109.7)
- added ?: , VIA, F.Cu at (99.6, 109.5)
- added ?: , VIA, F.Cu at (100.8, 109.7)
- added ?: , VIA, F.Cu at (102.0, 109.5)
- added ?: , VIA, F.Cu at (87.1, 104.7)
- added ?: , VIA, F.Cu at (93.7, 102.5)
- added ?: , VIA, F.Cu at (96.0, 104.8)
- added ?: , VIA, F.Cu at (92.5, 104.7)
- added ?: , VIA, F.Cu at (94.2, 108.5)
- added ?: , VIA, F.Cu at (127.1, 100.9)
- added ?: , VIA, F.Cu at (97.1, 109.5)
- added ?: , VIA, F.Cu at (97.1, 107.2)
- added ?: , VIA, F.Cu at (90.2, 102.5)
- added ?: , VIA, F.Cu at (86.3, 83.5)
- added ?: , VIA, F.Cu at (79.3, 92.8)
- added ?: , VIA, F.Cu at (88.4, 83.5)
- added ?: , VIA, F.Cu at (91.0, 83.5)
- added ?: , VIA, F.Cu at (103.3, 88.4)
- added ?: , VIA, F.Cu at (103.3, 90.2)
- added ?: , VIA, F.Cu at (96.9, 83.8)
- added ?: , VIA, F.Cu at (128.4, 103.8)
- added ?: , VIA, F.Cu at (98.8, 83.6)
- added ?: , VIA, F.Cu at (102.0, 90.2)
- added ?: , VIA, F.Cu at (102.0, 93.3)
- added ?: , VIA, F.Cu at (99.6, 93.3)
- added ?: , VIA, F.Cu at (100.8, 93.3)
- added ?: , VIA, F.Cu at (103.3, 93.3)
- added ?: , VIA, F.Cu at (98.3, 93.3)
- added ?: , VIA, F.Cu at (84.7, 95.2)
- added ?: , VIA, F.Cu at (84.0, 101.0)
- added ?: , VIA, F.Cu at (97.1, 95.3)
- added ?: , VIA, F.Cu at (132.1, 100.3)
- added ?: , VIA, F.Cu at (90.7, 95.1)
- added ?: , VIA, F.Cu at (90.7, 97.3)
- added ?: , VIA, F.Cu at (90.7, 101.0)
- added ?: , VIA, F.Cu at (90.7, 99.7)
- added ?: , VIA, F.Cu at (90.7, 98.5)
- added ?: , VIA, F.Cu at (92.5, 98.5)
- added ?: , VIA, F.Cu at (94.2, 99.7)
- added ?: , VIA, F.Cu at (92.5, 101.0)
- added ?: , VIA, F.Cu at (94.2, 97.3)
- added ?: , VIA, F.Cu at (92.5, 96.0)
- moved ? 16.2 mm to (99.6, 111.0)
- moved ? 13.7 mm to (113.8, 98.6)
- moved ? 11.9 mm to (111.4, 115.0)
- moved ? 11.2 mm to (112.6, 99.8)
- moved ? 2.40 mm to (111.4, 101.0)
- moved C15 0.50 mm to (81.9, 123.9)
Connections:
- ? pad : (no net) -> GND (x2)
Routing:
- net N-0000067: track 182.3 -> 201.5 mm, vias 3 -> 5
- net +BATT: track 82.4 -> 91.9 mm
- net GND: track 13.7 -> 23.1 mm
- net N-0000085: track 14.2 -> 16.2 mm
- net N-0000084: track 5.37 -> 7.13 mm
- net N-0000092: track 6.53 -> 7.65 mm
- net N-0000062: track 2.91 -> 4.04 mm
- net /Keypad/KEYPAD_COL_1: track 146.7 -> 145.6 mm
