File: Hardware/RevC/AriCalculator-RevC.kicad_pcb (KiCad board)
At the start: 2 copper layers, 76.2 x 147.3 mm, 414 parts, among them CON1 BDM, CON2 SPI, CON3 USB-MINI-B, IC1 MC9S12G, IC2 MCP1640, IC3 FT232RL, IC4 MCP1643, SW1 POWER SWITCH

Commit message: work in progress
Parts:
- moved ? 0.29 mm to (119.2, 93.8)
Changed lines of the file:
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@@
   )
   (module VIA (layer F.Cu)
-    (at 118.95 93.75)
+    (at 119.225 93.825)
     (fp_text reference "" (at 0 0) (layer F.SilkS) hide
       (effects (font (size 0.5 0.5) (thickness 0.125)))

Commit message: work in progress
Parts:
- removed the ? at (105.3, 128.6)
- removed the ? at (131.6, 125.2)
- removed the ? at (89.2, 135.6)
- added ?: , VIA, F.Cu at (87.7, 138.4)
- added ?: , VIA, F.Cu at (107.8, 138.3)
- added ?: , VIA, F.Cu at (104.5, 128.6)
- added ?: , VIA, F.Cu at (101.6, 134.6)
- added ?: , VIA, F.Cu at (91.4, 134.6)
- added ?: , VIA, F.Cu at (101.6, 154.9)
- added ?: , VIA, F.Cu at (121.3, 124.5)
- added ?: , VIA, F.Cu at (117.8, 128.2)
- added ?: , VIA, F.Cu at (112.8, 127.4)
- added ?: , VIA, F.Cu at (112.8, 123.0)
- added ?: , VIA, F.Cu at (119.8, 130.4)
- added ?: , VIA, F.Cu at (116.4, 124.5)
- added ?: , VIA, F.Cu at (117.3, 130.8)
- added ?: , VIA, F.Cu at (107.6, 131.0)
- added ?: , VIA, F.Cu at (122.7, 130.0)
- added ?: , VIA, F.Cu at (106.0, 128.6)
- added ?: , VIA, F.Cu at (99.5, 131.2)
- added ?: , VIA, F.Cu at (95.5, 130.8)
- added ?: , VIA, F.Cu at (91.4, 154.9)
- added ?: , VIA, F.Cu at (111.8, 154.9)
- added ?: , VIA, F.Cu at (132.1, 154.9)
- added ?: , VIA, F.Cu at (81.3, 154.9)
- added ?: , VIA, F.Cu at (132.1, 134.6)
- added ?: , VIA, F.Cu at (131.7, 125.2)
- added ?: , VIA, F.Cu at (82.8, 131.7)
- added ?: , VIA, F.Cu at (81.3, 134.6)
- added ?: , VIA, F.Cu at (121.9, 154.9)
- added ?: , VIA, F.Cu at (132.1, 144.8)
- added ?: , VIA, F.Cu at (81.3, 144.8)
- added ?: , VIA, F.Cu at (81.3, 165.1)
- added ?: , VIA, F.Cu at (132.1, 165.1)
- added ?: , VIA, F.Cu at (119.4, 165.1)
- added ?: , VIA, F.Cu at (94.0, 165.1)
- added ?: , VIA, F.Cu at (106.7, 165.1)
- added ? (x2): , VIA, F.Cu at (81.3, 175.3)
- added ?: , VIA, F.Cu at (83.5, 112.3)
- added ? (x2): , VIA, F.Cu at (132.1, 175.3)
- added ? (x2): , VIA, F.Cu at (119.4, 175.3)
- added ? (x2): , VIA, F.Cu at (94.0, 175.3)
- added ? (x2): , VIA, F.Cu at (106.7, 175.3)
- added ?: , VIA, F.Cu at (106.7, 185.4)
- added ?: , VIA, F.Cu at (84.5, 119.7)
- added ?: , VIA, F.Cu at (94.0, 185.4)
- added ?: , VIA, F.Cu at (119.4, 185.4)
- added ?: , VIA, F.Cu at (132.1, 185.4)
- added ?: , VIA, F.Cu at (81.3, 185.4)
- added ?: , VIA, F.Cu at (113.9, 131.2)
- added ?: , VIA, F.Cu at (81.3, 195.6)
- added ?: , VIA, F.Cu at (132.1, 195.6)
- added ?: , VIA, F.Cu at (119.4, 195.6)
- added ?: , VIA, F.Cu at (94.0, 195.6)
- added ?: , VIA, F.Cu at (106.7, 195.6)
- added ?: , VIA, F.Cu at (86.4, 131.7)
- added ?: , VIA, F.Cu at (83.4, 128.2)
- added ?: , VIA, F.Cu at (81.9, 93.8)
- added ?: , VIA, F.Cu at (134.0, 104.3)
- moved ? 8.42 mm to (92.5, 130.4)
- moved ? 3.83 mm to (102.8, 131.4)
- moved ? 1.64 mm to (93.9, 95.2)
- moved ? 1.36 mm to (134.0, 92.8)
- moved ? 0.39 mm to (126.5, 130.6)
- moved ? 0.10 mm to (108.7, 128.6)
Routing:
- net GND: track 23.1 -> 27.4 mm
- net /Keypad/KEYPAD_COL_2: track 137.3 -> 135.2 mm
- net /Keypad/KEYPAD_COL_0: track 154.1 -> 152.7 mm
- net /Keypad/KEYPAD_COL_3: track 155.4 -> 156.6 mm
- net /Keypad/KEYPAD_COL_5: track 124.0 -> 122.9 mm
- net /Keypad/KEYPAD_COL_4: track 181.1 -> 180.3 mm
- net VUSB: track 16.3 -> 17.2 mm
- net /Keypad/KEYPAD_COL_1: track 145.6 -> 144.8 mm
Other:
- board text added: "BDM"
- board text added: "BUSY"
- board text added: "ERROR"
- board text added: "OFF"
- board text added: "ON"
- board text added: "RX/TX"
- board text added: "SPI"

Commit message: work in progress
Parts:
- added ?: , via, F.Cu at (103.3, 101.0)
- added ?: , via, F.Cu at (99.6, 101.0)
- added ?: , via, F.Cu at (102.0, 101.0)
- added ?: , via, F.Cu at (99.6, 124.9)
- added ?: , via, F.Cu at (112.8, 125.1)
- added ?: , via, F.Cu at (124.1, 128.1)
- added ?: , via, F.Cu at (100.8, 101.0)
- added ?: , via, F.Cu at (125.8, 109.5)
- added ?: , via, F.Cu at (98.4, 101.0)
- added ?: , via, F.Cu at (115.1, 107.7)
- ? (x323): footprint VIA -> via
- C13: value 1uf -> 1uF
- DISP1: footprint DOGL128-6 -> dogl128-6
- KEY_A0, KEY_A1, KEY_A2, KEY_A3, KEY_A4, KEY_B0, KEY_B1, KEY_B2, KEY_B3, KEY_B4, KEY_C0, KEY_C1, KEY_C2, KEY_C3, KEY_C4, KEY_D0, KEY_D1, KEY_D2, KEY_D3, KEY_D4, KEY_E0, KEY_E1, KEY_E2, KEY_E3, KEY_E4, KEY_E5, KEY_F0, KEY_F1, KEY_F2, KEY_F3, KEY_F4, KEY_F5, KEY_G0, KEY_G1, KEY_G2, KEY_G3, KEY_G4, KEY_G5: footprint KEY -> key
- LED1, LED2, LED3: footprint Led_0805 -> led_0805
- LED10, LED11, LED12, LED13, LED14, LED15, LED16, LED17, LED18, LED19, LED20, LED21, LED4, LED5, LED6, LED7, LED8, LED9: footprint Led_1206 -> led_1206
- SG (x12): renamed from spark_gap_pad_0.8; value SG -> 0.8
- SG (x9): renamed from spark_gap_pad_1.0; value SG -> 1.0
- SG (x17): renamed from spark_gap_pad_0.6; value SG -> 0.6
- enclosure: value VAL** -> AriCalculator
- moved ? 8.35 mm to (115.1, 116.3)
Other:
- board text added: "+"
- board text added: "-"
- board text added: "0"
- board text added: "1"
- board text added: "2"
- board text added: "3"
- board text added: "4"
- board text added: "5"
- board text added: "A"
- board text added: "B"
- board text added: "C"
- board text added: "D"
- board text added: "E"
- board text added: "F"
- board text added: "G"
- board text added: "S12G"

Commit message: work in progress
Parts:
- added ?: , via, F.Cu at (124.2, 113.2)
- added ?: , via, F.Cu at (111.8, 87.0)
- added ?: , via, F.Cu at (115.1, 128.2)
- added ?: , via, F.Cu at (82.4, 87.0)
- added ?: , via, F.Cu at (113.8, 103.2)
- added ?: , via, F.Cu at (95.9, 87.8)
- added ?: , via, F.Cu at (99.6, 104.4)
- added ?: , via, F.Cu at (115.1, 102.7)
- added ?: , via, F.Cu at (102.0, 104.4)
- added ?: , via, F.Cu at (100.8, 104.4)
- added ?: , via, F.Cu at (112.6, 103.7)
- added ?: , via, F.Cu at (112.9, 91.5)
- added ?: , via, F.Cu at (98.4, 104.4)
- added ?: , via, F.Cu at (93.9, 88.4)
- added ?: , via, F.Cu at (92.0, 89.0)
- added ?: , via, F.Cu at (103.3, 104.4)
- added ?: , via, F.Cu at (120.0, 101.1)
- added ?: , via, F.Cu at (106.7, 104.5)
- added ?: , via, F.Cu at (110.1, 104.1)
- added ?: , via, F.Cu at (117.9, 100.9)
- added ?: , via, F.Cu at (97.1, 104.4)
- added ?: , via, F.Cu at (100.8, 85.7)
- added ?: , via, F.Cu at (122.8, 126.3)
- added ?: , via, F.Cu at (83.5, 126.5)
- added ?: , via, F.Cu at (123.8, 101.0)
- added ?: , via, F.Cu at (111.4, 103.9)
- added ?: , via, F.Cu at (116.3, 124.5)
- added ?: , via, F.Cu at (122.0, 116.8)
- added ?: , via, F.Cu at (97.8, 87.2)
- added G***: LOGO, logo_silk_CC-BY-SA_10x4.5mm, B.Cu at (116.3, 102.2)
- moved ? 0.98 mm to (96.0, 83.4)
Other:
- board text added: "AriCalculator"
- board text added: "Dirk Heisswolf 2014"
- board text added: "RevC"
- board text added: "http://hotwolf.github.io/AriCalculator"

Commit message: work in progress
Parts:
- BAT1, BAT2: footprint AAA-BATTERY -> AAA-battery
Changed lines of the file:
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@@
     )
   )
-  (module AAA-BATTERY (layer B.Cu)
-    (at 106.7 200.4)
-    (fp_text reference BAT2 (at 0 10.5) (layer B.SilkS)
-      (effects (font (size 1 1) (thickness 0.15)) (justify mirror))
-    )
-    (fp_text value AAA-BATTERY (at 0 5) (layer B.SilkS)
-      (effects (font (size 1 1) (thickness 0.15)) (justify mirror))
-    )
-    (fp_line (start 25.5 13) (end -25.5 13) (layer B.SilkS) (width 0.15))
-    (fp_line (start -25.5 13) (end -25.5 0) (layer B.SilkS) (width 0.15))
-    (fp_line (start -25.5 0) (end 25.5 0) (layer B.SilkS) (width 0.15))
-    (fp_line (start 25.5 0) (end 25.5 13) (layer B.SilkS) (width 0.15))
-    (pad 2 thru_hole rect (at 28 6.5) (size 3 5) (drill 0.5 (offset -1 0))
-      (layers *.Cu *.Mask B.SilkS)
-      (net 29 GND)
-      (zone_connect 1)
-      (thermal_width 1)
-    )
-    (pad 1 thru_hole rect (at -28 6.5 180) (size 3 5) (drill 0.5 (offset -1 0))
-      (layers *.Cu *.Mask B.SilkS)
-      (net 71 N-0000094)
-    )
-    (model 3D-Models/AAA-Battery.wrl
-      (at (xyz 0 0 -0.08))
-      (scale (xyz 1 1 1))
-      (rotate (xyz 0 0 0))
-    )
-  )
-  (module AAA-BATTERY (layer B.Cu)
-    (at 106.7 79 180)
-    (fp_text reference BAT1 (at 0 10.5 180) (layer B.SilkS)
-      (effects (font (size 1 1) (thickness 0.15)) (justify mirror))
-    )
-    (fp_text value AAA-BATTERY (at 0 5 180) (layer B.SilkS)
-      (effects (font (size 1 1) (thickness 0.15)) (justify mirror))
-    )
-    (fp_line (start 25.5 13) (end -25.5 13) (layer B.SilkS) (width 0.15))
-    (fp_line (start -25.5 13) (end -25.5 0) (layer B.SilkS) (width 0.15))
-    (fp_line (start -25.5 0) (end 25.5 0) (layer B.SilkS) (width 0.15))
-    (fp_line (start 25.5 0) (end 25.5 13) (layer B.SilkS) (width 0.15))
-    (pad 2 thru_hole rect (at 28 6.5 180) (size 3 5) (drill 0.5 (offset -1 0))
-      (layers *.Cu *.Mask B.SilkS)
-      (net 71 N-0000094)
-    )
-    (pad 1 thru_hole rect (at -28 6.5) (size 3 5) (drill 0.5 (offset -1 0))
-      (layers *.Cu *.Mask B.SilkS)
-      (net 70 N-0000093)
-    )
-    (model 3D-Models/AAA-Battery.wrl
-      (at (xyz 0 0 -0.08))
-      (scale (xyz 1 1 1))
-      (rotate (xyz 0 0 0))
-    )
-  )
   (module led_1206 (layer F.Cu)
     (at 120 103.4 180)
@@
       (xy 3.92176 -0.64516)) (layer B.SilkS) (width 0.00254))
   )
+  (module AAA-battery (layer B.Cu)
+    (at 106.7 79 180)
+    (fp_text reference BAT1 (at 0 10.5 180) (layer B.SilkS)
+      (effects (font (size 1 1) (thickness 0.15)) (justify mirror))
+    )
+    (fp_text value AAA-BATTERY (at 0 5 180) (layer B.SilkS)
+      (effects (font (size 1 1) (thickness 0.15)) (justify mirror))
+    )
+    (pad 2 thru_hole rect (at 28 6.5 180) (size 3 5) (drill 0.5 (offset -1 0))
+      (layers *.Cu *.Mask B.SilkS)
+      (net 71 N-0000094)
+    )
+    (pad 1 thru_hole rect (at -28 6.5) (size 3 5) (drill 0.5 (offset -1 0))
+      (layers *.Cu *.Mask B.SilkS)
+      (net 70 N-0000093)
+    )
+    (model 3D-Models/AAA-Battery.wrl
+      (at (xyz 0 0 0))
+      (scale (xyz 1 1 1))
+      (rotate (xyz 0 0 0))
+    )
+  )
+  (module AAA-battery (layer B.Cu)
+    (at 106.7 200.4)
+    (fp_text reference BAT2 (at 0 10.5) (layer B.SilkS)
+      (effects (font (size 1 1) (thickness 0.15)) (justify mirror))
+    )
+    (fp_text value AAA-BATTERY (at 0 5) (layer B.SilkS)
+      (effects (font (size 1 1) (thickness 0.15)) (justify mirror))
+    )
+    (pad 2 thru_hole rect (at 28 6.5) (size 3 5) (drill 0.5 (offset -1 0))
+      (layers *.Cu *.Mask B.SilkS)
+      (net 29 GND)
+    )
+    (pad 1 thru_hole rect (at -28 6.5 180) (size 3 5) (drill 0.5 (offset -1 0))
+      (layers *.Cu *.Mask B.SilkS)
+      (net 71 N-0000094)
+    )
+    (model 3D-Models/AAA-Battery.wrl
+      (at (xyz 0 0 0))
+      (scale (xyz 1 1 1))
+      (rotate (xyz 0 0 0))
+    )
+  )
   (gr_text http://hotwolf.github.io/AriCalculator (at 105.95 106.95) (layer B.SilkS)
